File: Designdocs/InhalerCapDevelopmentBoard.brd (EAGLE design)
At the start: 50.5 x 63.5 mm, 23 parts

Commit message: Rev. 1 of board
Parts:
- R6: value (none) -> 220
Routing:
- net N$14: track 58.2 -> 60.7 mm
- net N$2: track 120.9 -> 123.1 mm
- net N$22: track 38.1 -> 40.2 mm
- net N$13: track 52.2 -> 54.1 mm
- net N$15: track 52.5 -> 54.2 mm
- net N$21: track 38.3 -> 39.7 mm
- net GND: track 162.8 -> 163.9 mm
Other:
- board text added: "Discover"
- board text added: "Inhaler Cap Developement Board rev. 1"
- board text added: "Inhaler Use"
- board text added: "Power"
- board text added: "Reset"
- board text added: "Source"
